Commit message: adapted urdf with reduced number of collision joint and split of feet colliders

File: urdf/anymal.urdf (robot description, URDF)
Before this commit: robot anymal, 96 links, 95 joints
Links:
- removed link inspection_payload_camera
- removed link inspection_payload_camera_default
- removed link inspection_payload_head
- removed link inspection_payload_light
- removed link inspection_payload_microphone
- removed link inspection_payload_mount
- removed link inspection_payload_pan
- removed link inspection_payload_thermal_camera
- removed link inspection_payload_tilt
- added link hatch, mass 0.09653; visual mesh filename=package://anymal_d_simple_description/meshes/hatch.dae scale=1.0 1.0 1.0
- link LF_FOOT: geometry collision sphere radius=0.031455; visual mesh filename=package://anymal_d_simple_description/meshes/foot.dae scale=1.0 1.0 1.0
- link LF_HFE_drive: geometry visual mesh filename=package://anymal_d_simple_description/meshes/drive.dae scale=1.0 1.0 1.0
- link LF_KFE_drive: geometry visual mesh filename=package://anymal_d_simple_description/meshes/drive.dae scale=1.0 1.0 1.0
- link LF_shank_fixed: geometry collision cylinder length=0.39572 radius=0.0175; visual mesh filename=package://anymal_d_simple_description/meshes/shank_l.dae scale=1.0 1.0 1.0
- link LF_thigh_fixed: geometry collision box size=0.093 0.063 0.285; collision cylinder length=0.16313000000000001 radius=0.07
- link LH_FOOT: geometry collision sphere radius=0.031455; visual mesh filename=package://anymal_d_simple_description/meshes/foot.dae scale=1.0 1.0 1.0
- link LH_HFE_drive: geometry visual mesh filename=package://anymal_d_simple_description/meshes/drive.dae scale=1.0 1.0 1.0
- link LH_KFE_drive: geometry visual mesh filename=package://anymal_d_simple_description/meshes/drive.dae scale=1.0 1.0 1.0
- link LH_shank_fixed: geometry collision cylinder length=0.39572 radius=0.0175; visual mesh filename=package://anymal_d_simple_description/meshes/shank_r.dae scale=1.0 1.0 1.0
- link LH_thigh_fixed: geometry collision box size=0.093 0.063 0.285; collision cylinder length=0.16313000000000001 radius=0.07
- link RF_FOOT: geometry collision sphere radius=0.031455; visual mesh filename=package://anymal_d_simple_description/meshes/foot.dae scale=1.0 1.0 1.0
- link RF_HFE_drive: geometry visual mesh filename=package://anymal_d_simple_description/meshes/drive.dae scale=1.0 1.0 1.0
- link RF_KFE_drive: geometry visual mesh filename=package://anymal_d_simple_description/meshes/drive.dae scale=1.0 1.0 1.0
- link RF_shank_fixed: geometry collision cylinder length=0.39572 radius=0.0175; visual mesh filename=package://anymal_d_simple_description/meshes/shank_r.dae scale=1.0 1.0 1.0
- link RF_thigh_fixed: geometry collision box size=0.093 0.063 0.285; collision cylinder length=0.16313000000000001 radius=0.07
- link RH_FOOT: geometry collision sphere radius=0.031455; visual mesh filename=package://anymal_d_simple_description/meshes/foot.dae scale=1.0 1.0 1.0
- link RH_HFE_drive: geometry visual mesh filename=package://anymal_d_simple_description/meshes/drive.dae scale=1.0 1.0 1.0
- link RH_KFE_drive: geometry visual mesh filename=package://anymal_d_simple_description/meshes/drive.dae scale=1.0 1.0 1.0
- link RH_shank_fixed: geometry collision cylinder length=0.39572 radius=0.0175; visual mesh filename=package://anymal_d_simple_description/meshes/shank_l.dae scale=1.0 1.0 1.0
- link RH_thigh_fixed: geometry collision box size=0.093 0.063 0.285; collision cylinder length=0.16313000000000001 radius=0.07
- link base: geometry collision box size=0.894 0.1615 0.356; visual mesh filename=package://anymal_d_simple_description/meshes/base.dae scale=1.0 1.0 1.0
- link lidar: geometry visual mesh filename=package://anymal_d_simple_description/meshes/lidar.dae; visual mesh filename=package://anymal_d_simple_description/meshes/lidar_guard.dae
Joints:
- removed joint base_to_inspection_payload_mount
- removed joint inspection_payload_head_to_camera
- removed joint inspection_payload_head_to_light
- removed joint inspection_payload_head_to_microphone
- removed joint inspection_payload_head_to_thermal_camera
- removed joint inspection_payload_mount_to_camera_default
- removed joint inspection_payload_mount_to_pan
- removed joint inspection_payload_pan_to_tilt
- removed joint inspection_payload_tilt_to_head
- added joint base_to_hatch: type fixed, parent base, child hatch, origin xyz=0.14253 0.0 0.092 rpy=0 0 0

Commit message: removes base inertial link

File: urdf/anymal.urdf (robot description, URDF)
Before this commit: robot anymal, 88 links, 87 joints
Links:
- removed link base_inertia
- link base: mass None -> 8.27629
Joints:
- removed joint base_to_base_inertia
